File: boost_power.sch (KiCad schematic (older format))
At the start: 7 parts

Commit message: update pcb
Parts:
- C1: renamed from C?; value C -> 100uF; footprint (none) -> Capacitor_SMD:C_1210_3225Metric
- C2: renamed from C?; value C -> 10uF; footprint (none) -> Capacitor_SMD:C_1210_3225Metric
- D1: renamed from D?; footprint (none) -> Diode_SMD:D_1206_3216Metric
- J1, J2: renamed from J?; footprint (none) -> Connector_PinHeader_2.54mm:PinHeader_1x02_P2.54mm_Vertical
- L1: renamed from L?; footprint (none) -> Inductor_SMD:L_Bourns-SRN4018
- U1: renamed from U?; footprint SOT95P275X110-5N -> Package_TO_SOT_SMD:SOT-23-5; symbol NCP1400ASN33T1G:NCP1400ASN33T1G -> boost_power-rescue:NCP1400ASN33T1G-NCP1400ASN33T1G
Changed lines of the file:
@@
 EESchema Schematic File Version 4
+LIBS:boost_power-cache
 EELAYER 30 0
 EELAYER END
@@
 $EndDescr
 $Comp
-L NCP1400ASN33T1G:NCP1400ASN33T1G U?
+L boost_power-rescue:NCP1400ASN33T1G-NCP1400ASN33T1G U1
 U 1 1 5E33CB67
 P 4950 2700
-F 0 "U?" H 4950 3170 50  0000 C CNN
+F 0 "U1" H 4950 3170 50  0000 C CNN
 F 1 "NCP1400ASN33T1G" H 4950 3079 50  0000 C CNN
-F 2 "SOT95P275X110-5N" H 4950 2700 50  0001 L BNN
+F 2 "Package_TO_SOT_SMD:SOT-23-5" H 4950 2700 50  0001 L BNN
 F 3 "Unavailable" H 4950 2700 50  0001 L BNN
 F 4 "None" H 4950 2700 50  0001 L BNN "Поле4"
@@
 $EndComp
 $Comp
-L power:GND #PWR?
+L power:GND #PWR0101
 U 1 1 5E33D276
 P 4250 3100
-F 0 "#PWR?" H 4250 2850 50  0001 C CNN
+F 0 "#PWR0101" H 4250 2850 50  0001 C CNN
 F 1 "GND" H 4255 2927 50  0000 C CNN
 F 2 "" H 4250 3100 50  0001 C CNN
@@
 $EndComp
 $Comp
-L power:+1V2 #PWR?
+L power:+1V2 #PWR0102
 U 1 1 5E33D878
 P 3700 2250
-F 0 "#PWR?" H 3700 2100 50  0001 C CNN
+F 0 "#PWR0102" H 3700 2100 50  0001 C CNN
 F 1 "+1V2" H 3715 2423 50  0000 C CNN
 F 2 "" H 3700 2250 50  0001 C CNN
@@
 $EndComp
 $Comp
-L power:+3.3V #PWR?
+L power:+3.3V #PWR0103
 U 1 1 5E33E3B9
 P 6900 2250
-F 0 "#PWR?" H 6900 2100 50  0001 C CNN
+F 0 "#PWR0103" H 6900 2100 50  0001 C CNN
 F 1 "+3.3V" H 6915 2423 50  0000 C CNN
 F 2 "" H 6900 2250 50  0001 C CNN
@@
 $EndComp
 $Comp
-L Device:D_Schottky D?
+L Device:D_Schottky D1
 U 1 1 5E33EEA6
 P 6400 2250
-F 0 "D?" H 6400 2466 50  0000 C CNN
+F 0 "D1" H 6400 2466 50  0000 C CNN
 F 1 "D_Schottky" H 6400 2375 50  0000 C CNN
-F 2 "" H 6400 2250 50  0001 C CNN
+F 2 "Diode_SMD:D_1206_3216Metric" H 6400 2250 50  0001 C CNN
 F 3 "~" H 6400 2250 50  0001 C CNN
 	1    6400 2250
@@
 $EndComp
 $Comp
-L Device:C C?
+L Device:C C2
 U 1 1 5E34848C
 P 6750 2400
-F 0 "C?" H 6865 2446 50  0000 L CNN
-F 1 "C" H 6865 2355 50  0000 L CNN
-F 2 "" H 6788 2250 50  0001 C CNN
+F 0 "C2" H 6865 2446 50  0000 L CNN
+F 1 "10uF" H 6865 2355 50  0000 L CNN
+F 2 "Capacitor_SMD:C_1210_3225Metric" H 6788 2250 50  0001 C CNN
 F 3 "~" H 6750 2400 50  0001 C CNN
 	1    6750 2400
@@
 $EndComp
 $Comp
-L power:GND #PWR?
+L power:GND #PWR0104
 U 1 1 5E348EC2
 P 6750 2550
-F 0 "#PWR?" H 6750 2300 50  0001 C CNN
+F 0 "#PWR0104" H 6750 2300 50  0001 C CNN
 F 1 "GND" H 6755 2377 50  0000 C CNN
 F 2 "" H 6750 2550 50  0001 C CNN
@@
 $EndComp
 $Comp
-L power:GND #PWR?
+L power:GND #PWR0105
 U 1 1 5E3493CC
 P 3850 2550
-F 0 "#PWR?" H 3850 2300 50  0001 C CNN
+F 0 "#PWR0105" H 3850 2300 50  0001 C CNN
 F 1 "GND" H 3855 2377 50  0000 C CNN
 F 2 "" H 3850 2550 50  0001 C CNN
@@
 $EndComp
 $Comp
-L Device:C C?
+L Device:C C1
 U 1 1 5E349F83
 P 3850 2400
-F 0 "C?" H 3965 2446 50  0000 L CNN
-F 1 "C" H 3965 2355 50  0000 L CNN
-F 2 "" H 3888 2250 50  0001 C CNN
+F 0 "C1" H 3965 2446 50  0000 L CNN
+F 1 "100uF" H 3965 2355 50  0000 L CNN
+F 2 "Capacitor_SMD:C_1210_3225Metric" H 3888 2250 50  0001 C CNN
 F 3 "~" H 3850 2400 50  0001 C CNN
 	1    3850 2400
@@
 	3700 2250 3850 2250
 $Comp
-L pspice:INDUCTOR L?
+L pspice:INDUCTOR L1
 U 1 1 5E351F58
 P 4950 2050
-F 0 "L?" H 4950 2265 50  0000 C CNN
+F 0 "L1" H 4950 2265 50  0000 C CNN
 F 1 "INDUCTOR" H 4950 2174 50  0000 C CNN
-F 2 "" H 4950 2050 50  0001 C CNN
+F 2 "Inductor_SMD:L_Bourns-SRN4018" H 4950 2050 50  0001 C CNN
 F 3 "~" H 4950 2050 50  0001 C CNN
 	1    4950 2050
@@
 	5850 2050 6050 2050
 $Comp
-L Connector:Conn_01x02_Male J?
+L Connector:Conn_01x02_Male J2
 U 1 1 5E357E80
 P 7800 2350
-F 0 "J?" H 7772 2324 50  0000 R CNN
+F 0 "J2" H 7772 2324 50  0000 R CNN
 F 1 "Conn_01x02_Male" H 7772 2233 50  0000 R CNN
-F 2 "" H 7800 2350 50  0001 C CNN
+F 2 "Connector_PinHeader_2.54mm:PinHeader_1x02_P2.54mm_Vertical" H 7800 2350 50  0001 C CNN
 F 3 "~" H 7800 2350 50  0001 C CNN
 	1    7800 2350
@@
 $EndComp
 $Comp
-L Connector:Conn_01x02_Male J?
+L Connector:Conn_01x02_Male J1
 U 1 1 5E358D5E
 P 2950 2300
-F 0 "J?" H 3058 2481 50  0000 C CNN
+F 0 "J1" H 3058 2481 50  0000 C CNN
 F 1 "Conn_01x02_Male" H 3058 2390 50  0000 C CNN
-F 2 "" H 2950 2300 50  0001 C CNN
+F 2 "Connector_PinHeader_2.54mm:PinHeader_1x02_P2.54mm_Vertical" H 2950 2300 50  0001 C CNN
 F 3 "~" H 2950 2300 50  0001 C CNN
 	1    2950 2300
@@
 $EndComp
 $Comp
-L power:GND #PWR?
+L power:GND #PWR0106
 U 1 1 5E35A58D
 P 3150 2400
-F 0 "#PWR?" H 3150 2150 50  0001 C CNN
+F 0 "#PWR0106" H 3150 2150 50  0001 C CNN
 F 1 "GND" H 3155 2227 50  0000 C CNN
 F 2 "" H 3150 2400 50  0001 C CNN
@@
 $EndComp
 $Comp
-L power:GND #PWR?
+L power:GND #PWR0107
 U 1 1 5E35AEEA
 P 7600 2450
-F 0 "#PWR?" H 7600 2200 50  0001 C CNN
+F 0 "#PWR0107" H 7600 2200 50  0001 C CNN
 F 1 "GND" H 7605 2277 50  0000 C CNN
 F 2 "" H 7600 2450 50  0001 C CNN
@@
 $EndComp
 $Comp
-L power:+3.3V #PWR?
+L power:+3.3V #PWR0108
 U 1 1 5E35CC4A
 P 7600 2350
-F 0 "#PWR?" H 7600 2200 50  0001 C CNN
+F 0 "#PWR0108" H 7600 2200 50  0001 C CNN
 F 1 "+3.3V" H 7615 2523 50  0000 C CNN
 F 2 "" H 7600 2350 50  0001 C CNN
@@
 $EndComp
 $Comp
-L power:+1V2 #PWR?
+L power:+1V2 #PWR0109
 U 1 1 5E35D4C9
 P 3150 2300
-F 0 "#PWR?" H 3150 2150 50  0001 C CNN
+F 0 "#PWR0109" H 3150 2150 50  0001 C CNN
 F 1 "+1V2" H 3165 2473 50  0000 C CNN
 F 2 "" H 3150 2300 50  0001 C CNN
